Commit message: feat: 가제보 연결 성공
move_group_sim.launch.py >> move_group 서버 역시 use_sim_time:=true 로 설정이 되어야 함.

File: src/A1_URDF_description/urdf/A1_URDF.xacro (robot description, xacro)
@@ -2,6 +2,6 @@
 <robot name="A1_URDF" xmlns:xacro="http://www.ros.org/wiki/xacro">
   <xacro:include filename="$(find A1_URDF_description)/urdf/materials.xacro" />
-  <xacro:include filename="$(find A1_URDF_description)/urdf/A1_URDF.trans" />
-  <xacro:include filename="$(find A1_URDF_description)/urdf/A1_URDF.gazebo" />
+  <!-- <xacro:include filename="$(find A1_URDF_description)/urdf/A1_URDF.trans" /> -->
+  <!-- <xacro:include filename="$(find A1_URDF_description)/urdf/A1_URDF.gazebo" /> -->
   <link name="base_link">
     <inertial>
@@ -13,5 +13,5 @@
       <origin xyz="0 0 0" rpy="0 0 0"/>
       <geometry>
-        <mesh filename="package://A1_URDF_description/meshes/base_link.stl" scale="0.001 0.001 0.001"/>
+        <mesh filename="$(find A1_URDF_description)/meshes/base_link.stl" scale="0.001 0.001 0.001"/>
       </geometry>
       <material name="silver"/>
@@ -20,5 +20,5 @@
       <origin xyz="0 0 0" rpy="0 0 0"/>
       <geometry>
-        <mesh filename="package://A1_URDF_description/meshes/base_link.stl" scale="0.001 0.001 0.001"/>
+        <mesh filename="$(find A1_URDF_description)/meshes/base_link.stl" scale="0.001 0.001 0.001"/>
       </geometry>
     </collision>
@@ -33,5 +33,5 @@
       <origin xyz="-0.060809 -0.0785 -0.693" rpy="0 0 0"/>
       <geometry>
-        <mesh filename="package://A1_URDF_description/meshes/shoulder_pitch_link_1.stl" scale="0.001 0.001 0.001"/>
+        <mesh filename="$(find A1_URDF_description)/meshes/shoulder_pitch_link_1.stl" scale="0.001 0.001 0.001"/>
       </geometry>
       <material name="silver"/>
@@ -40,5 +40,5 @@
       <origin xyz="-0.060809 -0.0785 -0.693" rpy="0 0 0"/>
       <geometry>
-        <mesh filename="package://A1_URDF_description/meshes/shoulder_pitch_link_1.stl" scale="0.001 0.001 0.001"/>
+        <mesh filename="$(find A1_URDF_description)/meshes/shoulder_pitch_link_1.stl" scale="0.001 0.001 0.001"/>
       </geometry>
     </collision>
@@ -53,5 +53,5 @@
       <origin xyz="-0.042809 -0.1285 -0.693" rpy="0 0 0"/>
       <geometry>
-        <mesh filename="package://A1_URDF_description/meshes/shoulder_roll_link_1.stl" scale="0.001 0.001 0.001"/>
+        <mesh filename="$(find A1_URDF_description)/meshes/shoulder_roll_link_1.stl" scale="0.001 0.001 0.001"/>
       </geometry>
       <material name="silver"/>
@@ -60,5 +60,5 @@
       <origin xyz="-0.042809 -0.1285 -0.693" rpy="0 0 0"/>
       <geometry>
-        <mesh filename="package://A1_URDF_description/meshes/shoulder_roll_link_1.stl" scale="0.001 0.001 0.001"/>
+        <mesh filename="$(find A1_URDF_description)/meshes/shoulder_roll_link_1.stl" scale="0.001 0.001 0.001"/>
       </geometry>
     </collision>
@@ -73,5 +73,5 @@
       <origin xyz="-0.060809 -0.1285 -0.628" rpy="0 0 0"/>
       <geometry>
-        <mesh filename="package://A1_URDF_description/meshes/shoulder_yaw_link_1.stl" scale="0.001 0.001 0.001"/>
+        <mesh filename="$(find A1_URDF_description)/meshes/shoulder_yaw_link_1.stl" scale="0.001 0.001 0.001"/>
       </geometry>
       <material name="silver"/>
@@ -80,5 +80,5 @@
       <origin xyz="-0.060809 -0.1285 -0.628" rpy="0 0 0"/>
       <geometry>
-        <mesh filename="package://A1_URDF_description/meshes/shoulder_yaw_link_1.stl" scale="0.001 0.001 0.001"/>
+        <mesh filename="$(find A1_URDF_description)/meshes/shoulder_yaw_link_1.stl" scale="0.001 0.001 0.001"/>
       </geometry>
     </collision>
@@ -93,5 +93,5 @@
       <origin xyz="-0.060809 -0.102 -0.513" rpy="0 0 0"/>
       <geometry>
-        <mesh filename="package://A1_URDF_description/meshes/elbow_link_1.stl" scale="0.001 0.001 0.001"/>
+        <mesh filename="$(find A1_URDF_description)/meshes/elbow_link_1.stl" scale="0.001 0.001 0.001"/>
       </geometry>
       <material name="silver"/>
@@ -100,5 +100,5 @@
       <origin xyz="-0.060809 -0.102 -0.513" rpy="0 0 0"/>
       <geometry>
-        <mesh filename="package://A1_URDF_description/meshes/elbow_link_1.stl" scale="0.001 0.001 0.001"/>
+        <mesh filename="$(find A1_URDF_description)/meshes/elbow_link_1.stl" scale="0.001 0.001 0.001"/>
       </geometry>
     </collision>
@@ -113,5 +113,5 @@
       <origin xyz="-0.060809 -0.1285 -0.414" rpy="0 0 0"/>
       <geometry>
-        <mesh filename="package://A1_URDF_description/meshes/wrist_yaw_link_1.stl" scale="0.001 0.001 0.001"/>
+        <mesh filename="$(find A1_URDF_description)/meshes/wrist_yaw_link_1.stl" scale="0.001 0.001 0.001"/>
       </geometry>
       <material name="silver"/>
@@ -120,5 +120,5 @@
       <origin xyz="-0.060809 -0.1285 -0.414" rpy="0 0 0"/>
       <geometry>
-        <mesh filename="package://A1_URDF_description/meshes/wrist_yaw_link_1.stl" scale="0.001 0.001 0.001"/>
+        <mesh filename="$(find A1_URDF_description)/meshes/wrist_yaw_link_1.stl" scale="0.001 0.001 0.001"/>
       </geometry>
     </collision>
@@ -133,5 +133,5 @@
       <origin xyz="-0.085809 -0.1285 -0.323" rpy="0 0 0"/>
       <geometry>
-        <mesh filename="package://A1_URDF_description/meshes/wrist_pitch_link_1.stl" scale="0.001 0.001 0.001"/>
+        <mesh filename="$(find A1_URDF_description)/meshes/wrist_pitch_link_1.stl" scale="0.001 0.001 0.001"/>
       </geometry>
       <material name="silver"/>
@@ -140,5 +140,5 @@
       <origin xyz="-0.085809 -0.1285 -0.323" rpy="0 0 0"/>
       <geometry>
-        <mesh filename="package://A1_URDF_description/meshes/wrist_pitch_link_1.stl" scale="0.001 0.001 0.001"/>
+        <mesh filename="$(find A1_URDF_description)/meshes/wrist_pitch_link_1.stl" scale="0.001 0.001 0.001"/>
       </geometry>
     </collision>
@@ -153,5 +153,5 @@
       <origin xyz="-0.060809 -0.1505 -0.323" rpy="0 0 0"/>
       <geometry>
-        <mesh filename="package://A1_URDF_description/meshes/wrist_roll_link_1.stl" scale="0.001 0.001 0.001"/>
+        <mesh filename="$(find A1_URDF_description)/meshes/wrist_roll_link_1.stl" scale="0.001 0.001 0.001"/>
       </geometry>
       <material name="silver"/>
@@ -160,5 +160,5 @@
       <origin xyz="-0.060809 -0.1505 -0.323" rpy="0 0 0"/>
       <geometry>
-        <mesh filename="package://A1_URDF_description/meshes/wrist_roll_link_1.stl" scale="0.001 0.001 0.001"/>
+        <mesh filename="$(find A1_URDF_description)/meshes/wrist_roll_link_1.stl" scale="0.001 0.001 0.001"/>
       </geometry>
     </collision>

File: src/areum2_moveit_config/config/A1_URDF.ros2_control.xacro (robot description, xacro)
@@ -6,5 +6,6 @@
             <hardware>
                 <!-- By default, set up controllers for simulation. This won't work on real hardware -->
-                <plugin>mock_components/GenericSystem</plugin>
+                <!-- <plugin>mock_components/GenericSystem</plugin> -->
+                <plugin>gazebo_ros2_control/GazeboSystem</plugin>
             </hardware>
             <joint name="shoulder_pitch_joint">
@@ -58,4 +59,11 @@
             </joint>
         </ros2_control>
+        <gazebo>
+            <plugin name="gazebo_ros2_control" filename="libgazebo_ros2_control.so">
+                <parameters>$(find areum2_moveit_config)/config/ros2_controllers.yaml</parameters>
+                <robot_param>robot_description</robot_param>
+                <robot_param_node>robot_state_publisher</robot_param_node>
+            </plugin>
+        </gazebo>
     </xacro:macro>
 </robot>

File: src/areum2_moveit_config/config/A1_URDF.urdf.xacro (robot description, xacro)
@@ -6,4 +6,6 @@
     <!-- Import control_xacro -->
     <xacro:include filename="A1_URDF.ros2_control.xacro" />
+    <!-- Gazebo World Connect -->
+    <xacro:include filename="$(find areum2_moveit_config)/config/A1_URDF.gazebo_frame.xacro" />
     <xacro:A1_URDF_ros2_control name="FakeSystem" initial_positions_file="$(arg initial_positions_file)"/>
 </robot>

Commit message: feat: {최종} Gazebo <> Ros2 연결하기 위해 필요한 최소한의 파일구조를 정의함.
---

[src/A1_URDF_description/urdf/A1_URDF.xacro]
- A1_URDF_description 디렉토리에는 오로지 로봇의 형상정보만 담기도록 함.
  따라서 gazebo, trans 파일 참조는 제거.
- 또한 gazebo 가 visual, collision 을 참조할 수 있도록, find 명령을 씀.

[src/areum2_moveit_config/config/A1_URDF.ros2_control.xacro]
- gazebo 하드웨어 브릿지(?)를 plugin 형식으로 추가. (이게 뭔 역할을 하는지는 추후 공부 필요.)
- gazebo 가 ros2_controlllers.yaml 정보를 참조할 수 있게 함.

[src/areum2_moveit_config/config/A1_URDF.gazebo_frame.xacro]
- gazebo <> base_link 고정하기 위한 가상 fixed 조인트 생성.

[src/areum2_moveit_config/config/A1_URDF.urdf.xacro]
- 위에서 생성한 가상 fixed 조인트를 메인 URDF 에 호출.

[src/areum2_moveit_config/launch/move_group_sim.launch.py]
- move_group 서버 노드 역시, 시뮬레이션에서 사용되기 위해선 use_sim_time = true 가 되어야 함.
  그렇지 않으면, 요청 시간이 수십년의 시간으로 차이가 나버려 로봇의 joint states 를 서버가 불러오지를 못 함.
- use_sim_time 이 정확히 어떤 역할을 하는지 추후 공부 필요.
- 해당 launch 파일의 코드는 추후 공부 필요.

[src/areum2_moveit_config/package.xml]
- joint_trajectory_controller, gazebo_ros_control 패키지 include 함.
  마찬가지로 이 패키지들이 뭐하는 애들인지는 추후 공부 필요.

File: src/A1_URDF_description/urdf/A1_URDF.xacro (robot description, xacro)
@@ -2,6 +2,4 @@
 <robot name="A1_URDF" xmlns:xacro="http://www.ros.org/wiki/xacro">
   <xacro:include filename="$(find A1_URDF_description)/urdf/materials.xacro" />
-  <xacro:include filename="$(find A1_URDF_description)/urdf/A1_URDF.trans" />
-  <xacro:include filename="$(find A1_URDF_description)/urdf/A1_URDF.gazebo" />
   <link name="base_link">
     <inertial>
@@ -13,5 +11,5 @@
       <origin xyz="0 0 0" rpy="0 0 0"/>
       <geometry>
-        <mesh filename="package://A1_URDF_description/meshes/base_link.stl" scale="0.001 0.001 0.001"/>
+        <mesh filename="$(find A1_URDF_description)/meshes/base_link.stl" scale="0.001 0.001 0.001"/>
       </geometry>
       <material name="silver"/>
@@ -20,5 +18,5 @@
       <origin xyz="0 0 0" rpy="0 0 0"/>
       <geometry>
-        <mesh filename="package://A1_URDF_description/meshes/base_link.stl" scale="0.001 0.001 0.001"/>
+        <mesh filename="$(find A1_URDF_description)/meshes/base_link.stl" scale="0.001 0.001 0.001"/>
       </geometry>
     </collision>
@@ -33,5 +31,5 @@
       <origin xyz="-0.060809 -0.0785 -0.693" rpy="0 0 0"/>
       <geometry>
-        <mesh filename="package://A1_URDF_description/meshes/shoulder_pitch_link_1.stl" scale="0.001 0.001 0.001"/>
+        <mesh filename="$(find A1_URDF_description)/meshes/shoulder_pitch_link_1.stl" scale="0.001 0.001 0.001"/>
       </geometry>
       <material name="silver"/>
@@ -40,5 +38,5 @@
       <origin xyz="-0.060809 -0.0785 -0.693" rpy="0 0 0"/>
       <geometry>
-        <mesh filename="package://A1_URDF_description/meshes/shoulder_pitch_link_1.stl" scale="0.001 0.001 0.001"/>
+        <mesh filename="$(find A1_URDF_description)/meshes/shoulder_pitch_link_1.stl" scale="0.001 0.001 0.001"/>
       </geometry>
     </collision>
@@ -53,5 +51,5 @@
       <origin xyz="-0.042809 -0.1285 -0.693" rpy="0 0 0"/>
       <geometry>
-        <mesh filename="package://A1_URDF_description/meshes/shoulder_roll_link_1.stl" scale="0.001 0.001 0.001"/>
+        <mesh filename="$(find A1_URDF_description)/meshes/shoulder_roll_link_1.stl" scale="0.001 0.001 0.001"/>
       </geometry>
       <material name="silver"/>
@@ -60,5 +58,5 @@
       <origin xyz="-0.042809 -0.1285 -0.693" rpy="0 0 0"/>
       <geometry>
-        <mesh filename="package://A1_URDF_description/meshes/shoulder_roll_link_1.stl" scale="0.001 0.001 0.001"/>
+        <mesh filename="$(find A1_URDF_description)/meshes/shoulder_roll_link_1.stl" scale="0.001 0.001 0.001"/>
       </geometry>
     </collision>
@@ -73,5 +71,5 @@
       <origin xyz="-0.060809 -0.1285 -0.628" rpy="0 0 0"/>
       <geometry>
-        <mesh filename="package://A1_URDF_description/meshes/shoulder_yaw_link_1.stl" scale="0.001 0.001 0.001"/>
+        <mesh filename="$(find A1_URDF_description)/meshes/shoulder_yaw_link_1.stl" scale="0.001 0.001 0.001"/>
       </geometry>
       <material name="silver"/>
@@ -80,5 +78,5 @@
       <origin xyz="-0.060809 -0.1285 -0.628" rpy="0 0 0"/>
       <geometry>
-        <mesh filename="package://A1_URDF_description/meshes/shoulder_yaw_link_1.stl" scale="0.001 0.001 0.001"/>
+        <mesh filename="$(find A1_URDF_description)/meshes/shoulder_yaw_link_1.stl" scale="0.001 0.001 0.001"/>
       </geometry>
     </collision>
@@ -93,5 +91,5 @@
       <origin xyz="-0.060809 -0.102 -0.513" rpy="0 0 0"/>
       <geometry>
-        <mesh filename="package://A1_URDF_description/meshes/elbow_link_1.stl" scale="0.001 0.001 0.001"/>
+        <mesh filename="$(find A1_URDF_description)/meshes/elbow_link_1.stl" scale="0.001 0.001 0.001"/>
       </geometry>
       <material name="silver"/>
@@ -100,5 +98,5 @@
       <origin xyz="-0.060809 -0.102 -0.513" rpy="0 0 0"/>
       <geometry>
-        <mesh filename="package://A1_URDF_description/meshes/elbow_link_1.stl" scale="0.001 0.001 0.001"/>
+        <mesh filename="$(find A1_URDF_description)/meshes/elbow_link_1.stl" scale="0.001 0.001 0.001"/>
       </geometry>
     </collision>
@@ -113,5 +111,5 @@
       <origin xyz="-0.060809 -0.1285 -0.414" rpy="0 0 0"/>
       <geometry>
-        <mesh filename="package://A1_URDF_description/meshes/wrist_yaw_link_1.stl" scale="0.001 0.001 0.001"/>
+        <mesh filename="$(find A1_URDF_description)/meshes/wrist_yaw_link_1.stl" scale="0.001 0.001 0.001"/>
       </geometry>
       <material name="silver"/>
@@ -120,5 +118,5 @@
       <origin xyz="-0.060809 -0.1285 -0.414" rpy="0 0 0"/>
       <geometry>
-        <mesh filename="package://A1_URDF_description/meshes/wrist_yaw_link_1.stl" scale="0.001 0.001 0.001"/>
+        <mesh filename="$(find A1_URDF_description)/meshes/wrist_yaw_link_1.stl" scale="0.001 0.001 0.001"/>
       </geometry>
     </collision>
@@ -133,5 +131,5 @@
       <origin xyz="-0.085809 -0.1285 -0.323" rpy="0 0 0"/>
       <geometry>
-        <mesh filename="package://A1_URDF_description/meshes/wrist_pitch_link_1.stl" scale="0.001 0.001 0.001"/>
+        <mesh filename="$(find A1_URDF_description)/meshes/wrist_pitch_link_1.stl" scale="0.001 0.001 0.001"/>
       </geometry>
       <material name="silver"/>
@@ -140,5 +138,5 @@
       <origin xyz="-0.085809 -0.1285 -0.323" rpy="0 0 0"/>
       <geometry>
-        <mesh filename="package://A1_URDF_description/meshes/wrist_pitch_link_1.stl" scale="0.001 0.001 0.001"/>
+        <mesh filename="$(find A1_URDF_description)/meshes/wrist_pitch_link_1.stl" scale="0.001 0.001 0.001"/>
       </geometry>
     </collision>
@@ -153,5 +151,5 @@
       <origin xyz="-0.060809 -0.1505 -0.323" rpy="0 0 0"/>
       <geometry>
-        <mesh filename="package://A1_URDF_description/meshes/wrist_roll_link_1.stl" scale="0.001 0.001 0.001"/>
+        <mesh filename="$(find A1_URDF_description)/meshes/wrist_roll_link_1.stl" scale="0.001 0.001 0.001"/>
       </geometry>
       <material name="silver"/>
@@ -160,5 +158,5 @@
       <origin xyz="-0.060809 -0.1505 -0.323" rpy="0 0 0"/>
       <geometry>
-        <mesh filename="package://A1_URDF_description/meshes/wrist_roll_link_1.stl" scale="0.001 0.001 0.001"/>
+        <mesh filename="$(find A1_URDF_description)/meshes/wrist_roll_link_1.stl" scale="0.001 0.001 0.001"/>
       </geometry>
     </collision>

File: src/areum2_moveit_config/config/A1_URDF.ros2_control.xacro (robot description, xacro)
@@ -6,5 +6,7 @@
             <hardware>
                 <!-- By default, set up controllers for simulation. This won't work on real hardware -->
-                <plugin>mock_components/GenericSystem</plugin>
+                <!-- <plugin>mock_components/GenericSystem</plugin> -->
+                <!-- For Gazebo to ros2_control Bridge -->
+                <plugin>gazebo_ros2_control/GazeboSystem</plugin>
             </hardware>
             <joint name="shoulder_pitch_joint">
@@ -58,4 +60,9 @@
             </joint>
         </ros2_control>
+        <gazebo>
+            <plugin name="gazebo_ros2_control" filename="libgazebo_ros2_control.so">
+                <parameters>$(find areum2_moveit_config)/config/ros2_controllers.yaml</parameters>
+            </plugin>
+        </gazebo>
     </xacro:macro>
 </robot>

File: src/areum2_moveit_config/config/A1_URDF.urdf.xacro (robot description, xacro)
@@ -6,4 +6,6 @@
     <!-- Import control_xacro -->
     <xacro:include filename="A1_URDF.ros2_control.xacro" />
+    <!-- [Gazebo World <> Robot] Fixed Connect -->
+    <xacro:include filename="$(find areum2_moveit_config)/config/A1_URDF.gazebo_frame.xacro" />
     <xacro:A1_URDF_ros2_control name="FakeSystem" initial_positions_file="$(arg initial_positions_file)"/>
 </robot>
