Commit message: feat: (추가) Gazebo <> Ros2 연결되기 위한 조건들 추가 작성
[기존 문제]
A1_URDF_description 디렉토리에 있던 xacro 의 visual, collision 을 move_group 노드가 인식하지 못 하던 문제가 발생

[해결 방법]
xacro 파일의 visual, collision 태그를 모두, find 명령이 아닌, 기존 디폴트 방식으로 되어있던 package:// 방식으로 변경하였더니,
move_group 이 다시 visual, collision 을 잘 import 하는 것을 발견함.

하지만 이 경우 gazebo 가 import 를 하지 못하는 문제가 이어서 발생하였음.
이를 해결하기 위해, 다음 두 파일을 수정하였음.

---

[src/A1_URDF_description/urdf/A1_URDF.xacro]

visual 과 collision 의 geometry 의 mesh 를 다시 package:// 방식으로 하여 move_group 이 이 매쉬를 참조할 수 있도록 함.

[src/A1_URDF_description/package.xml]

<exec_depend>gazebo_ros</exec_depend>
    exec_depend 는 ros2 가 빌드 후 "실행할 때" 필요한 의존 패키지를 정의하는 부분이다.
    gazebo 는 ros가 "실행할 때" 불러와지기 때문에, exec_depend 에 정의를 한다.

<export>
    ...
    <gazebo_ros gazebo_model_path="${prefix}/.."/>
</export>
    ${prefix}의 의미: ROS 2 빌드 시스템(ament)이 이 패키지를 빌드한 최종 설치 경로
    (/home/junha/ws_arum2_ros2/install/A1_URDF_description/share/A1_URDF_description) 이다.
    /.. 가 붙었기에 상위로 한번 올라간 디렉토리 /share를 의미함.

    GAZEBO_MODEL_PATH: Gazebo에서 모델을 검색할 경로를 지정하는 변수
    gazebo_model_path 환경변수에 위 디렉토리를 대입하여, Gazebo 가 모델을 검색할 때 share 디렉토리 부터 검색을 할 수 있도록 지정하였다.

File: src/A1_URDF_description/urdf/A1_URDF.xacro (robot description, xacro)
@@ -11,5 +11,5 @@
       <origin xyz="0 0 0" rpy="0 0 0"/>
       <geometry>
-        <mesh filename="$(find A1_URDF_description)/meshes/base_link.stl" scale="0.001 0.001 0.001"/>
+        <mesh filename="package://A1_URDF_description/meshes/base_link.stl" scale="0.001 0.001 0.001"/>
       </geometry>
       <material name="silver"/>
@@ -18,5 +18,5 @@
       <origin xyz="0 0 0" rpy="0 0 0"/>
       <geometry>
-        <mesh filename="$(find A1_URDF_description)/meshes/base_link.stl" scale="0.001 0.001 0.001"/>
+        <mesh filename="package://A1_URDF_description/meshes/base_link.stl" scale="0.001 0.001 0.001"/>
       </geometry>
     </collision>
@@ -31,5 +31,5 @@
       <origin xyz="-0.060809 -0.0785 -0.693" rpy="0 0 0"/>
       <geometry>
-        <mesh filename="$(find A1_URDF_description)/meshes/shoulder_pitch_link_1.stl" scale="0.001 0.001 0.001"/>
+        <mesh filename="package://A1_URDF_description/meshes/shoulder_pitch_link_1.stl" scale="0.001 0.001 0.001"/>
       </geometry>
       <material name="silver"/>
@@ -38,5 +38,5 @@
       <origin xyz="-0.060809 -0.0785 -0.693" rpy="0 0 0"/>
       <geometry>
-        <mesh filename="$(find A1_URDF_description)/meshes/shoulder_pitch_link_1.stl" scale="0.001 0.001 0.001"/>
+        <mesh filename="package://A1_URDF_description/meshes/shoulder_pitch_link_1.stl" scale="0.001 0.001 0.001"/>
       </geometry>
     </collision>
@@ -51,5 +51,5 @@
       <origin xyz="-0.042809 -0.1285 -0.693" rpy="0 0 0"/>
       <geometry>
-        <mesh filename="$(find A1_URDF_description)/meshes/shoulder_roll_link_1.stl" scale="0.001 0.001 0.001"/>
+        <mesh filename="package://A1_URDF_description/meshes/shoulder_roll_link_1.stl" scale="0.001 0.001 0.001"/>
       </geometry>
       <material name="silver"/>
@@ -58,5 +58,5 @@
       <origin xyz="-0.042809 -0.1285 -0.693" rpy="0 0 0"/>
       <geometry>
-        <mesh filename="$(find A1_URDF_description)/meshes/shoulder_roll_link_1.stl" scale="0.001 0.001 0.001"/>
+        <mesh filename="package://A1_URDF_description/meshes/shoulder_roll_link_1.stl" scale="0.001 0.001 0.001"/>
       </geometry>
     </collision>
@@ -71,5 +71,5 @@
       <origin xyz="-0.060809 -0.1285 -0.628" rpy="0 0 0"/>
       <geometry>
-        <mesh filename="$(find A1_URDF_description)/meshes/shoulder_yaw_link_1.stl" scale="0.001 0.001 0.001"/>
+        <mesh filename="package://A1_URDF_description/meshes/shoulder_yaw_link_1.stl" scale="0.001 0.001 0.001"/>
       </geometry>
       <material name="silver"/>
@@ -78,5 +78,5 @@
       <origin xyz="-0.060809 -0.1285 -0.628" rpy="0 0 0"/>
       <geometry>
-        <mesh filename="$(find A1_URDF_description)/meshes/shoulder_yaw_link_1.stl" scale="0.001 0.001 0.001"/>
+        <mesh filename="package://A1_URDF_description/meshes/shoulder_yaw_link_1.stl" scale="0.001 0.001 0.001"/>
       </geometry>
     </collision>
@@ -91,5 +91,5 @@
       <origin xyz="-0.060809 -0.102 -0.513" rpy="0 0 0"/>
       <geometry>
-        <mesh filename="$(find A1_URDF_description)/meshes/elbow_link_1.stl" scale="0.001 0.001 0.001"/>
+        <mesh filename="package://A1_URDF_description/meshes/elbow_link_1.stl" scale="0.001 0.001 0.001"/>
       </geometry>
       <material name="silver"/>
@@ -98,5 +98,5 @@
       <origin xyz="-0.060809 -0.102 -0.513" rpy="0 0 0"/>
       <geometry>
-        <mesh filename="$(find A1_URDF_description)/meshes/elbow_link_1.stl" scale="0.001 0.001 0.001"/>
+        <mesh filename="package://A1_URDF_description/meshes/elbow_link_1.stl" scale="0.001 0.001 0.001"/>
       </geometry>
     </collision>
@@ -111,5 +111,5 @@
       <origin xyz="-0.060809 -0.1285 -0.414" rpy="0 0 0"/>
       <geometry>
-        <mesh filename="$(find A1_URDF_description)/meshes/wrist_yaw_link_1.stl" scale="0.001 0.001 0.001"/>
+        <mesh filename="package://A1_URDF_description/meshes/wrist_yaw_link_1.stl" scale="0.001 0.001 0.001"/>
       </geometry>
       <material name="silver"/>
@@ -118,5 +118,5 @@
       <origin xyz="-0.060809 -0.1285 -0.414" rpy="0 0 0"/>
       <geometry>
-        <mesh filename="$(find A1_URDF_description)/meshes/wrist_yaw_link_1.stl" scale="0.001 0.001 0.001"/>
+        <mesh filename="package://A1_URDF_description/meshes/wrist_yaw_link_1.stl" scale="0.001 0.001 0.001"/>
       </geometry>
     </collision>
@@ -131,5 +131,5 @@
       <origin xyz="-0.085809 -0.1285 -0.323" rpy="0 0 0"/>
       <geometry>
-        <mesh filename="$(find A1_URDF_description)/meshes/wrist_pitch_link_1.stl" scale="0.001 0.001 0.001"/>
+        <mesh filename="package://A1_URDF_description/meshes/wrist_pitch_link_1.stl" scale="0.001 0.001 0.001"/>
       </geometry>
       <material name="silver"/>
@@ -138,5 +138,5 @@
       <origin xyz="-0.085809 -0.1285 -0.323" rpy="0 0 0"/>
       <geometry>
-        <mesh filename="$(find A1_URDF_description)/meshes/wrist_pitch_link_1.stl" scale="0.001 0.001 0.001"/>
+        <mesh filename="package://A1_URDF_description/meshes/wrist_pitch_link_1.stl" scale="0.001 0.001 0.001"/>
       </geometry>
     </collision>
@@ -151,5 +151,5 @@
       <origin xyz="-0.060809 -0.1505 -0.323" rpy="0 0 0"/>
       <geometry>
-        <mesh filename="$(find A1_URDF_description)/meshes/wrist_roll_link_1.stl" scale="0.001 0.001 0.001"/>
+        <mesh filename="package://A1_URDF_description/meshes/wrist_roll_link_1.stl" scale="0.001 0.001 0.001"/>
       </geometry>
       <material name="silver"/>
@@ -158,5 +158,5 @@
       <origin xyz="-0.060809 -0.1505 -0.323" rpy="0 0 0"/>
       <geometry>
-        <mesh filename="$(find A1_URDF_description)/meshes/wrist_roll_link_1.stl" scale="0.001 0.001 0.001"/>
+        <mesh filename="package://A1_URDF_description/meshes/wrist_roll_link_1.stl" scale="0.001 0.001 0.001"/>
       </geometry>
     </collision>
