Commit message: feat: Octomap 통합 성공함.

File: src/areum2_moveit_config/config/A1_URDF.camera_frame.xacro (robot description, xacro)
@@ -4,5 +4,6 @@
     <parent link="world" />
     <child link="camera_link" />
-    <origin xyz="0.0 0.0 0.8" rpy="0 0 3.14159" />
+    <origin xyz="0.1 0.0 0.75" rpy="0 0.174533 0" />
+    <!-- pitch = 10deg 아래로 수그리게 함. -->
   </joint>
   <link name="camera_link" />
