Commit message: feat: B6 URDF 양팔 관절각도 부호 대칭되도록 <joint> 의 <axis> 부호 수정.

File: src/B6_description/urdf/B6.xacro (robot description, xacro)
@@ -346,5 +346,5 @@
   <parent link="base_link"/>
   <child link="shoulder_pitch_link_L_1"/>
-  <axis xyz="0.0 1.0 0.0"/>
+  <axis xyz="0.0 -1.0 0.0"/>
   <limit upper="3.141593" lower="-3.141593" effort="100" velocity="100"/>
 </joint>
@@ -356,9 +356,9 @@
   <limit upper="2.96706" lower="-0.261799" effort="100" velocity="100"/>
 </joint>
-<joint name="shouler_yaw_joint_L" type="revolute">
+<joint name="shoulder_yaw_joint_L" type="revolute">
   <origin xyz="0.02 0.0 -0.065" rpy="0 0 0"/>
   <parent link="shoulder_roll_link_L_1"/>
   <child link="shoulder_yaw_link_L_1"/>
-  <axis xyz="-0.0 -0.0 1.0"/>
+  <axis xyz="-0.0 -0.0 -1.0"/>
   <limit upper="1.396263" lower="-1.396263" effort="100" velocity="100"/>
 </joint>
@@ -367,5 +367,5 @@
   <parent link="shoulder_yaw_link_L_1"/>
   <child link="elbow_link_L_1"/>
-  <axis xyz="0.0 1.0 0.0"/>
+  <axis xyz="0.0 -1.0 0.0"/>
   <limit upper="0.872665" lower="-2.094395" effort="100" velocity="100"/>
 </joint>
@@ -374,5 +374,5 @@
   <parent link="elbow_link_L_1"/>
   <child link="wrist_roll_link_L_1"/>
-  <axis xyz="0.0 0.0 1.0"/>
+  <axis xyz="0.0 0.0 -1.0"/>
   <limit upper="1.745329" lower="-1.745329" effort="100" velocity="100"/>
 </joint>
@@ -381,5 +381,5 @@
   <parent link="wrist_roll_link_L_1"/>
   <child link="wrist_yaw_link_L_1"/>
-  <axis xyz="1.0 0.0 0.0"/>
+  <axis xyz="-1.0 0.0 0.0"/>
   <limit upper="0.523599" lower="-0.523599" effort="100" velocity="100"/>
 </joint>
@@ -388,5 +388,5 @@
   <parent link="wrist_yaw_link_L_1"/>
   <child link="wrist_pitch_link_L_1"/>
-  <axis xyz="-0.0 1.0 -0.0"/>
+  <axis xyz="-0.0 -1.0 -0.0"/>
   <limit upper="1.570796" lower="-1.570796" effort="100" velocity="100"/>
 </joint>
@@ -400,5 +400,5 @@
   <parent link="base_link"/>
   <child link="shoulder_pitch_link_R_1"/>
-  <axis xyz="0.0 1.0 0.0"/>
+  <axis xyz="0.0 -1.0 0.0"/>
   <limit upper="3.141593" lower="-3.141593" effort="100" velocity="100"/>
 </joint>
@@ -414,5 +414,5 @@
   <parent link="shoulder_yaw_link_R_1"/>
   <child link="elbow_link_R_1"/>
-  <axis xyz="0.0 1.0 0.0"/>
+  <axis xyz="0.0 -1.0 0.0"/>
   <limit upper="0.872665" lower="-2.094395" effort="100" velocity="100"/>
 </joint>
@@ -435,5 +435,5 @@
   <parent link="wrist_yaw_link_R_1"/>
   <child link="wrist_pitch_link_R_1"/>
-  <axis xyz="-0.0 1.0 -0.0"/>
+  <axis xyz="-0.0 -1.0 -0.0"/>
   <limit upper="1.570796" lower="-1.570796" effort="100" velocity="100"/>
 </joint>
@@ -447,5 +447,5 @@
   <parent link="shoulder_pitch_link_R_1"/>
   <child link="shoulder_roll_link_R_1"/>
-  <axis xyz="1.0 -0.0 0.0"/>
+  <axis xyz="-1.0 -0.0 0.0"/>
   <limit upper="0.261799" lower="-2.96706" effort="100" velocity="100"/>
 </joint>

Commit message: feat: B6 URDF 양팔 관절각도 부호 대칭되도록 <joint> 의 부호 수정후, 각도 한계도 수정.

File: src/B6_description/urdf/B6.xacro (robot description, xacro)
@@ -368,5 +368,5 @@
   <child link="elbow_link_L_1"/>
   <axis xyz="0.0 -1.0 0.0"/>
-  <limit upper="0.872665" lower="-2.094395" effort="100" velocity="100"/>
+  <limit upper="2.094395" lower="-0.872665" effort="100" velocity="100"/>
 </joint>
 <joint name="wrist_roll_joint_L" type="revolute">
@@ -415,5 +415,5 @@
   <child link="elbow_link_R_1"/>
   <axis xyz="0.0 -1.0 0.0"/>
-  <limit upper="0.872665" lower="-2.094395" effort="100" velocity="100"/>
+  <limit upper="2.094395" lower="-0.872665" effort="100" velocity="100"/>
 </joint>
 <joint name="wrist_roll_joint_R" type="revolute">
@@ -448,5 +448,5 @@
   <child link="shoulder_roll_link_R_1"/>
   <axis xyz="-1.0 -0.0 0.0"/>
-  <limit upper="0.261799" lower="-2.96706" effort="100" velocity="100"/>
+  <limit upper="2.96706" lower="-0.261799" effort="100" velocity="100"/>
 </joint>
 </robot>
