Commit message: feat: 리얼 하드웨어 테스트 용으로 shoulder_pitch_r, elbow_r 을 리얼 하드웨어 interface 쪽으로 연결함.

File: src/areumii_moveit_config/config/B6.ros2_control.xacro (robot description, xacro)
@@ -3,5 +3,6 @@
     <xacro:macro name="B6_ros2_control" params="name initial_positions_file">
         <xacro:property name="initial_positions" value="${load_yaml(initial_positions_file)['initial_positions']}"/>
-        <ros2_control name="${name}" type="system">
+        <ros2_control name="Test_can_interface" type="system">
+            <!-- 테스트용으로 두 joint 만 실제 hardware interface 로 분리해놓음 -->
             <hardware>
                 <!-- By default, set up controllers for simulation. This won't work on real hardware -->
@@ -20,4 +21,22 @@
                 <state_interface name="velocity"/>
             </joint>
+            <joint name="elbow_joint_R">
+                <command_interface name="position"/>
+                <command_interface name="velocity"/>
+                <state_interface name="position">
+                  <param name="initial_value">${initial_positions['elbow_joint_R']}</param>
+                </state_interface>
+                <state_interface name="velocity"/>
+            </joint>
+        </ros2_control>
+        <ros2_control name="${name}" type="system">
+            <hardware>
+                <!-- By default, set up controllers for simulation. This won't work on real hardware -->
+                <plugin>mock_components/GenericSystem</plugin>
+                <!-- For Gazebo to ros2_control Bridge -->
+                <!-- <plugin>gazebo_ros2_control/GazeboSystem</plugin> -->
+                <!-- For Real Hardware interface -->
+                <!-- <plugin>areumii_hardware_interface/AreumiiHardwareInterface</plugin> -->
+            </hardware>
             <joint name="shoulder_roll_joint_R">
                 <command_interface name="position"/>
@@ -33,12 +52,4 @@
                 <state_interface name="position">
                   <param name="initial_value">${initial_positions['shoulder_yaw_joint_R']}</param>
-                </state_interface>
-                <state_interface name="velocity"/>
-            </joint>
-            <joint name="elbow_joint_R">
-                <command_interface name="position"/>
-                <command_interface name="velocity"/>
-                <state_interface name="position">
-                  <param name="initial_value">${initial_positions['elbow_joint_R']}</param>
                 </state_interface>
                 <state_interface name="velocity"/>

Commit message: feat: isaacsim 에 B6 import 하는것 성공함.
TODO
- isaacsim 에서 omni graph 의 articulation root 를 B6로 하게될때 오류나는거 해결해여함

File: src/areumii_moveit_config/config/B6.ros2_control.xacro (robot description, xacro)
@@ -3,6 +3,5 @@
     <xacro:macro name="B6_ros2_control" params="name initial_positions_file">
         <xacro:property name="initial_positions" value="${load_yaml(initial_positions_file)['initial_positions']}"/>
-        <ros2_control name="Test_can_interface" type="system">
-            <!-- 테스트용으로 두 joint 만 실제 hardware interface 로 분리해놓음 -->
+        <ros2_control name="${name}" type="system">
             <hardware>
                 <!-- By default, set up controllers for simulation. This won't work on real hardware -->
@@ -11,5 +10,9 @@
                 <!-- <plugin>gazebo_ros2_control/GazeboSystem</plugin> -->
                 <!-- For Real Hardware interface -->
-                <plugin>areumii_hardware_interface/AreumiiHardwareInterface</plugin>
+                <!-- <plugin>areumii_hardware_interface/AreumiiHardwareInterface</plugin> -->
+                <!-- For Isaac Sim to ros2_control Bridge -->
+                <plugin>topic_based_ros2_control/TopicBasedSystem</plugin>
+                <param name="joint_commands_topic">/isaac_joint_commands</param>
+                <param name="joint_states_topic">/isaac_joint_states</param>
             </hardware>
             <joint name="shoulder_pitch_joint_R">
@@ -21,22 +24,4 @@
                 <state_interface name="velocity"/>
             </joint>
-            <joint name="elbow_joint_R">
-                <command_interface name="position"/>
-                <command_interface name="velocity"/>
-                <state_interface name="position">
-                  <param name="initial_value">${initial_positions['elbow_joint_R']}</param>
-                </state_interface>
-                <state_interface name="velocity"/>
-            </joint>
-        </ros2_control>
-        <ros2_control name="${name}" type="system">
-            <hardware>
-                <!-- By default, set up controllers for simulation. This won't work on real hardware -->
-                <plugin>mock_components/GenericSystem</plugin>
-                <!-- For Gazebo to ros2_control Bridge -->
-                <!-- <plugin>gazebo_ros2_control/GazeboSystem</plugin> -->
-                <!-- For Real Hardware interface -->
-                <!-- <plugin>areumii_hardware_interface/AreumiiHardwareInterface</plugin> -->
-            </hardware>
             <joint name="shoulder_roll_joint_R">
                 <command_interface name="position"/>
@@ -52,4 +37,12 @@
                 <state_interface name="position">
                   <param name="initial_value">${initial_positions['shoulder_yaw_joint_R']}</param>
+                </state_interface>
+                <state_interface name="velocity"/>
+            </joint>
+            <joint name="elbow_joint_R">
+                <command_interface name="position"/>
+                <command_interface name="velocity"/>
+                <state_interface name="position">
+                  <param name="initial_value">${initial_positions['elbow_joint_R']}</param>
                 </state_interface>
                 <state_interface name="velocity"/>

Commit message: feat: 오른쪽 팔 모터 전체 구동 성공. (EE 제외)

File: src/areumii_moveit_config/config/B6.ros2_control.xacro (robot description, xacro)
@@ -13,4 +13,12 @@
                 <plugin>areumii_hardware_interface/AreumiiHardwareInterface</plugin>
             </hardware>
+            <joint name="shoulder_roll_joint_R">
+                <command_interface name="position"/>
+                <command_interface name="velocity"/>
+                <state_interface name="position">
+                  <param name="initial_value">${initial_positions['shoulder_roll_joint_R']}</param>
+                </state_interface>
+                <state_interface name="velocity"/>
+            </joint>
             <joint name="shoulder_pitch_joint_R">
                 <command_interface name="position"/>
@@ -21,4 +29,12 @@
                 <state_interface name="velocity"/>
             </joint>
+            <joint name="shoulder_yaw_joint_R">
+                <command_interface name="position"/>
+                <command_interface name="velocity"/>
+                <state_interface name="position">
+                  <param name="initial_value">${initial_positions['shoulder_yaw_joint_R']}</param>
+                </state_interface>
+                <state_interface name="velocity"/>
+            </joint>
             <joint name="elbow_joint_R">
                 <command_interface name="position"/>
@@ -26,30 +42,4 @@
                 <state_interface name="position">
                   <param name="initial_value">${initial_positions['elbow_joint_R']}</param>
-                </state_interface>
-                <state_interface name="velocity"/>
-            </joint>
-        </ros2_control>
-        <ros2_control name="${name}" type="system">
-            <hardware>
-                <!-- By default, set up controllers for simulation. This won't work on real hardware -->
-                <plugin>mock_components/GenericSystem</plugin>
-                <!-- For Gazebo to ros2_control Bridge -->
-                <!-- <plugin>gazebo_ros2_control/GazeboSystem</plugin> -->
-                <!-- For Real Hardware interface -->
-                <!-- <plugin>areumii_hardware_interface/AreumiiHardwareInterface</plugin> -->
-            </hardware>
-            <joint name="shoulder_roll_joint_R">
-                <command_interface name="position"/>
-                <command_interface name="velocity"/>
-                <state_interface name="position">
-                  <param name="initial_value">${initial_positions['shoulder_roll_joint_R']}</param>
-                </state_interface>
-                <state_interface name="velocity"/>
-            </joint>
-            <joint name="shoulder_yaw_joint_R">
-                <command_interface name="position"/>
-                <command_interface name="velocity"/>
-                <state_interface name="position">
-                  <param name="initial_value">${initial_positions['shoulder_yaw_joint_R']}</param>
                 </state_interface>
                 <state_interface name="velocity"/>
@@ -79,4 +69,14 @@
                 <state_interface name="velocity"/>
             </joint>
+        </ros2_control>
+        <ros2_control name="${name}" type="system">
+            <hardware>
+                <!-- By default, set up controllers for simulation. This won't work on real hardware -->
+                <plugin>mock_components/GenericSystem</plugin>
+                <!-- For Gazebo to ros2_control Bridge -->
+                <!-- <plugin>gazebo_ros2_control/GazeboSystem</plugin> -->
+                <!-- For Real Hardware interface -->
+                <!-- <plugin>areumii_hardware_interface/AreumiiHardwareInterface</plugin> -->
+            </hardware>
             <joint name="shoulder_pitch_joint_L">
                 <command_interface name="position"/>

Commit message: feat: shoulder_pitch, shoulder_roll 순서에 맞게 수정.

File: src/areumii_moveit_config/config/B6.ros2_control.xacro (robot description, xacro)
@@ -13,4 +13,12 @@
                 <plugin>areumii_hardware_interface/AreumiiHardwareInterface</plugin>
             </hardware>
+            <joint name="shoulder_pitch_joint_R">
+                <command_interface name="position"/>
+                <command_interface name="velocity"/>
+                <state_interface name="position">
+                  <param name="initial_value">${initial_positions['shoulder_pitch_joint_R']}</param>
+                </state_interface>
+                <state_interface name="velocity"/>
+            </joint>
             <joint name="shoulder_roll_joint_R">
                 <command_interface name="position"/>
@@ -18,12 +26,4 @@
                 <state_interface name="position">
                   <param name="initial_value">${initial_positions['shoulder_roll_joint_R']}</param>
-                </state_interface>
-                <state_interface name="velocity"/>
-            </joint>
-            <joint name="shoulder_pitch_joint_R">
-                <command_interface name="position"/>
-                <command_interface name="velocity"/>
-                <state_interface name="position">
-                  <param name="initial_value">${initial_positions['shoulder_pitch_joint_R']}</param>
                 </state_interface>
                 <state_interface name="velocity"/>
