Commit message: feat: 아이작 urdf 모델도 joint 거울 상에서, 모두 동일 상으로 바꿈

File: src/areumii_description/urdf/areumii.urdf (robot description, URDF)
Before this commit: robot areumii, 22 links, 21 joints
Joints:
- joint elbow_joint_L: axis 0.0 1.0 -0.0 -> 0.0 -1.0 -0.0; limit lower=-2.094395 upper=0.872665 effort=100 velocity=100 -> lower=-0.872665 upper=2.094395 effort=100 velocity=100
- joint elbow_joint_R: axis 0.0 1.0 -0.0 -> 0.0 -1.0 -0.0; limit lower=-2.094395 upper=0.872665 effort=100 velocity=100 -> lower=-0.872665 upper=2.094395 effort=100 velocity=100
- joint shoulder_roll_joint_R: axis 1.0 -0.0 0.0 -> -1.0 -0.0 0.0; limit lower=-2.96706 upper=0.261799 effort=100 velocity=100 -> lower=-0.261799 upper=2.96706 effort=100 velocity=100
- joint shouler_yaw_joint_L: axis 0.0 0.0 1.0 -> 0.0 0.0 -1.0
- joint wrist_pitch_joint_L: axis 0.0 1.0 -0.0 -> 0.0 -1.0 -0.0
- joint wrist_pitch_joint_R: axis 0.0 1.0 -0.0 -> 0.0 -1.0 -0.0
- joint wrist_roll_joint_L: axis 0.0 0.0 1.0 -> 0.0 0.0 -1.0
- joint wrist_yaw_joint_L: axis 1.0 -0.0 0.0 -> -1.0 -0.0 0.0
