Commit message: feat: C1 양팔 joint 구동시 부호가 대칭이 되도록 회전축과 각도한계 재지정.
[수정한 부분들]
shoulder roll R
shoulder yaw L
elbow (둘다 반대방향으로)
wrist roll L
wrist pitch (둘다 반대방향으로)
wrist yaw L

File: src/areumii_description/urdf/areumii.xacro (robot description, xacro)
@@ -435,5 +435,5 @@
   <parent link="shoulder_roll_link_L_1"/>
   <child link="shoulder_yaw_link_L_1"/>
-  <axis xyz="0.0 0.0 1.0"/>
+  <axis xyz="0.0 0.0 -1.0"/>
   <limit upper="1.396263" lower="-1.396263" effort="100" velocity="100"/>
 </joint>
@@ -442,6 +442,6 @@
   <parent link="shoulder_yaw_link_L_1"/>
   <child link="elbow_link_L_1"/>
-  <axis xyz="0.0 1.0 -0.0"/>
-  <limit upper="0.872665" lower="-2.094395" effort="100" velocity="100"/>
+  <axis xyz="0.0 -1.0 -0.0"/>
+  <limit upper="2.094395" lower="-0.872665" effort="100" velocity="100"/>
 </joint>
 <joint name="wrist_roll_joint_L" type="revolute">
@@ -449,5 +449,5 @@
   <parent link="elbow_link_L_1"/>
   <child link="wrist_roll_link_L_1"/>
-  <axis xyz="0.0 0.0 1.0"/>
+  <axis xyz="0.0 0.0 -1.0"/>
   <limit upper="1.745329" lower="-1.745329" effort="100" velocity="100"/>
 </joint>
@@ -456,5 +456,5 @@
   <parent link="wrist_roll_link_L_1"/>
   <child link="wrist_yaw_link_L_1"/>
-  <axis xyz="1.0 -0.0 0.0"/>
+  <axis xyz="-1.0 -0.0 0.0"/>
   <limit upper="0.523599" lower="-0.523599" effort="100" velocity="100"/>
 </joint>
@@ -463,5 +463,5 @@
   <parent link="wrist_yaw_link_L_1"/>
   <child link="wrist_pitch_link_L_1"/>
-  <axis xyz="0.0 1.0 -0.0"/>
+  <axis xyz="0.0 -1.0 -0.0"/>
   <limit upper="1.570796" lower="-1.570796" effort="100" velocity="100"/>
 </joint>
@@ -477,6 +477,6 @@
   <parent link="shoulder_yaw_link_R_1"/>
   <child link="elbow_link_R_1"/>
-  <axis xyz="0.0 1.0 -0.0"/>
-  <limit upper="0.872665" lower="-2.094395" effort="100" velocity="100"/>
+  <axis xyz="0.0 -1.0 -0.0"/>
+  <limit upper="2.094395" lower="-0.872665" effort="100" velocity="100"/>
 </joint>
 <joint name="wrist_roll_joint_R" type="revolute">
@@ -498,5 +498,5 @@
   <parent link="wrist_yaw_link_R_1"/>
   <child link="wrist_pitch_link_R_1"/>
-  <axis xyz="0.0 1.0 -0.0"/>
+  <axis xyz="0.0 -1.0 -0.0"/>
   <limit upper="1.570796" lower="-1.570796" effort="100" velocity="100"/>
 </joint>
@@ -505,6 +505,6 @@
   <parent link="shoulder_pitch_link_R_1"/>
   <child link="shoulder_roll_link_R_1"/>
-  <axis xyz="1.0 -0.0 0.0"/>
-  <limit upper="0.261799" lower="-2.96706" effort="100" velocity="100"/>
+  <axis xyz="-1.0 -0.0 0.0"/>
+  <limit upper="2.96706" lower="-0.261799" effort="100" velocity="100"/>
 </joint>
 <joint name="shoulder_pitch_joint_R" type="revolute">

Commit message: feat: C1 의 joint 축방향들 모두 원상태로 방향 수정함

File: src/areumii_description/urdf/areumii.xacro (robot description, xacro)
@@ -435,5 +435,5 @@
   <parent link="shoulder_roll_link_L_1"/>
   <child link="shoulder_yaw_link_L_1"/>
-  <axis xyz="0.0 0.0 -1.0"/>
+  <axis xyz="0.0 0.0 1.0"/>
   <limit upper="1.396263" lower="-1.396263" effort="100" velocity="100"/>
 </joint>
@@ -442,6 +442,6 @@
   <parent link="shoulder_yaw_link_L_1"/>
   <child link="elbow_link_L_1"/>
-  <axis xyz="0.0 -1.0 -0.0"/>
-  <limit upper="2.094395" lower="-0.872665" effort="100" velocity="100"/>
+  <axis xyz="0.0 1.0 -0.0"/>
+  <limit upper="0.872665" lower="-2.094395" effort="100" velocity="100"/>
 </joint>
 <joint name="wrist_roll_joint_L" type="revolute">
@@ -449,5 +449,5 @@
   <parent link="elbow_link_L_1"/>
   <child link="wrist_roll_link_L_1"/>
-  <axis xyz="0.0 0.0 -1.0"/>
+  <axis xyz="0.0 0.0 1.0"/>
   <limit upper="1.745329" lower="-1.745329" effort="100" velocity="100"/>
 </joint>
@@ -456,5 +456,5 @@
   <parent link="wrist_roll_link_L_1"/>
   <child link="wrist_yaw_link_L_1"/>
-  <axis xyz="-1.0 -0.0 0.0"/>
+  <axis xyz="1.0 -0.0 0.0"/>
   <limit upper="0.523599" lower="-0.523599" effort="100" velocity="100"/>
 </joint>
@@ -463,5 +463,5 @@
   <parent link="wrist_yaw_link_L_1"/>
   <child link="wrist_pitch_link_L_1"/>
-  <axis xyz="0.0 -1.0 -0.0"/>
+  <axis xyz="0.0 1.0 -0.0"/>
   <limit upper="1.570796" lower="-1.570796" effort="100" velocity="100"/>
 </joint>
@@ -477,6 +477,6 @@
   <parent link="shoulder_yaw_link_R_1"/>
   <child link="elbow_link_R_1"/>
-  <axis xyz="0.0 -1.0 -0.0"/>
-  <limit upper="2.094395" lower="-0.872665" effort="100" velocity="100"/>
+  <axis xyz="0.0 1.0 -0.0"/>
+  <limit upper="0.872665" lower="-2.094395" effort="100" velocity="100"/>
 </joint>
 <joint name="wrist_roll_joint_R" type="revolute">
@@ -498,5 +498,5 @@
   <parent link="wrist_yaw_link_R_1"/>
   <child link="wrist_pitch_link_R_1"/>
-  <axis xyz="0.0 -1.0 -0.0"/>
+  <axis xyz="0.0 1.0 -0.0"/>
   <limit upper="1.570796" lower="-1.570796" effort="100" velocity="100"/>
 </joint>
@@ -505,6 +505,6 @@
   <parent link="shoulder_pitch_link_R_1"/>
   <child link="shoulder_roll_link_R_1"/>
-  <axis xyz="-1.0 -0.0 0.0"/>
-  <limit upper="2.96706" lower="-0.261799" effort="100" velocity="100"/>
+  <axis xyz="1.0 -0.0 0.0"/>
+  <limit upper="0.261799" lower="-2.96706" effort="100" velocity="100"/>
 </joint>
 <joint name="shoulder_pitch_joint_R" type="revolute">

Commit message: feat:
kinematics - 솔버 시간 여유조금 더줌.
sensors_3d - pointcloud 로 만들게끔 함(box 형태로 voxel 삭제 위함)
base_link_plate_removed - 아래 정판때문에 padding 되어 테이블 일부가 삭제되는문제 발생. 따라서 아래 정판 일부 매쉬를 제거함.
preprocessing.yaml - remove_table: true >> 이거랑 gpd.cpp 의 remove_table 이랑 어떻게 할지 정해야 함.

File: src/areumii_description/urdf/areumii.xacro (robot description, xacro)
@@ -11,5 +11,5 @@
     <origin xyz="0 0 0" rpy="0 0 0"/>
     <geometry>
-      <mesh filename="package://areumii_description/meshes/base_link.stl" scale="0.001 0.001 0.001"/>
+      <mesh filename="package://areumii_description/meshes/base_link_plate_removed.stl" scale="0.001 0.001 0.001"/>
     </geometry>
     <material name="silver"/>
@@ -18,5 +18,5 @@
     <origin xyz="0 0 0" rpy="0 0 0"/>
     <geometry>
-      <mesh filename="package://areumii_description/meshes/base_link.stl" scale="0.001 0.001 0.001"/>
+      <mesh filename="package://areumii_description/meshes/base_link_plate_removed.stl" scale="0.001 0.001 0.001"/>
     </geometry>
   </collision>
