Commit message: feat: camera_color_optical_frame 추가

File: src/areum_ii_moveit_config/config/areumii.camera_frame.xacro (robot description, xacro)
@@ -8,3 +8,12 @@
   </joint>
   <link name="camera_link"/>
+  <joint name="camera_link_to_color_optical_frame" type="fixed">
+    <parent link="camera_link"/>
+    <child link="camera_color_optical_frame"/>
+    <origin xyz="0 0.0148 0" rpy="-1.57079632679 0 -1.57079632679"/>
+    <!-- /camera/camera/aligned_depth_to_color/image_raw 와 /camera/camera/color/image_raw 데이터 모두 camera_color_optical_frame 에서 정의가 된다. -->
+    <!-- Left IR 에 위치한 camera_link 좌표계에서 camera_color_optical_frame 좌표계로 +y, 0.0148 만큼 차이가 나므로 origin 을 다음과 같이 수정한다. -->
+    <!-- [출처] https://github.com/realsenseai/realsense-ros -->
+  </joint>
+  <link name="camera_color_optical_frame"/>
 </robot>

Commit message: feat: C1 URDF에 Depth 카메라 마운트 설계수정된거 반영함

File: src/areum_ii_moveit_config/config/areumii.camera_frame.xacro (robot description, xacro)
@@ -4,5 +4,5 @@
     <parent link="base_link" />
     <child link="camera_link" />
-    <origin xyz="0.099303 0.017962 0.700916" rpy="0 1.04719755 0" />
+    <origin xyz="0.098803 0.017962 0.846782" rpy="0 1.04719755 0" />
     <!-- pitch = 60deg 아래로 수그리게 함. -->
   </joint>

File: src/areumii_description/urdf/areumii.urdf (robot description, URDF)
Before this commit: robot areumii, 22 links, 21 joints
Joints:
- joint base_link_to_camera_link: origin xyz=0.099303 0.017962 0.700916 rpy=0 1.04719755 0 -> xyz=0.098803 0.017962 0.846782 rpy=0 1.04719755 0
