Commit message: feat: isaac sim 에 C1 과 Depth 를 올리기 위한 설정 완료. 또한 demo.launch 실행 시 hardware type 을 launch argument 로 사용자가 지정할 수 있게끔 함.

File: src/areum_ii_moveit_config/config/areumii.ros2_control.xacro (robot description, xacro)
@@ -1,10 +1,19 @@
 <?xml version="1.0"?>
 <robot xmlns:xacro="http://www.ros.org/wiki/xacro">
-    <xacro:macro name="areumii_ros2_control" params="name initial_positions_file">
+    <xacro:macro name="areumii_ros2_control" params="name initial_positions_file ros2_control_hardware_type">
         <xacro:property name="initial_positions" value="${load_yaml(initial_positions_file)['initial_positions']}"/>
         <ros2_control name="${name}" type="system">
             <hardware>
-                <!-- By default, set up controllers for simulation. This won't work on real hardware -->
-                <plugin>mock_components/GenericSystem</plugin>
+                <xacro:if value="${ros2_control_hardware_type == 'mock_components'}">
+                  <plugin>mock_components/GenericSystem</plugin>
+                </xacro:if>
+                <xacro:if value="${ros2_control_hardware_type == 'real_hardware'}">
+                  <plugin>areumii_hardware_interface/AreumiiHardwareInterface</plugin>
+                </xacro:if>
+                <xacro:if value="${ros2_control_hardware_type == 'isaac'}">
+                  <plugin>topic_based_ros2_control/TopicBasedSystem</plugin>
+                  <param name="joint_commands_topic">/isaac_joint_commands</param>
+                  <param name="joint_states_topic">/isaac_joint_states</param>
+                </xacro:if>
             </hardware>
             <joint name="shoulder_pitch_joint_L">

File: src/areum_ii_moveit_config/config/areumii.urdf.xacro (robot description, xacro)
@@ -2,4 +2,5 @@
 <robot xmlns:xacro="http://www.ros.org/wiki/xacro" name="areumii">
     <xacro:arg name="initial_positions_file" default="initial_positions.yaml" />
+    <xacro:arg name="ros2_control_hardware_type" default="mock_components" />
     <!-- Import areumii urdf file -->
     <xacro:include filename="$(find areumii_description)/urdf/areumii.xacro" />
@@ -8,4 +9,4 @@
     <!-- [base_link > camera_link TF]  -->
     <xacro:include filename="areumii.camera_frame.xacro" />
-    <xacro:areumii_ros2_control name="FakeSystem" initial_positions_file="$(arg initial_positions_file)"/>
+    <xacro:areumii_ros2_control name="FakeSystem" initial_positions_file="$(arg initial_positions_file)" ros2_control_hardware_type="$(arg ros2_control_hardware_type)"/>
 </robot>

File: src/areumii_description/urdf/areumii.xacro (robot description, xacro)
@@ -2,6 +2,4 @@
 <robot name="areumii" xmlns:xacro="http://www.ros.org/wiki/xacro">
 <xacro:include filename="$(find areumii_description)/urdf/materials.xacro" />
-<xacro:include filename="$(find areumii_description)/urdf/areumii.trans" />
-<xacro:include filename="$(find areumii_description)/urdf/areumii.gazebo" />
 <link name="base_link">
   <inertial>
