Commit message: feat: dgl_ros 를 통해 grasp_poses 후보들 생성 완료. ros2 control 을 아이작, CAN 통신, mock 각각에 대해서 분기문으로 수정. C1 URDF joint 축들을 거울 상으로 다시 배치 함. actor.hpp 은 dgl_ros 액션 서버가 SUCCEED 상태로 반환 되도록 코드를 수정함.

File: src/areum_ii_moveit_config/config/areumii.ros2_control.xacro (robot description, xacro)
@@ -3,163 +3,464 @@
     <xacro:macro name="areumii_ros2_control" params="name initial_positions_file ros2_control_hardware_type">
         <xacro:property name="initial_positions" value="${load_yaml(initial_positions_file)['initial_positions']}"/>
-        <ros2_control name="${name}" type="system">
-            <hardware>
-                <xacro:if value="${ros2_control_hardware_type == 'mock_components'}">
-                  <plugin>mock_components/GenericSystem</plugin>
-                </xacro:if>
-                <xacro:if value="${ros2_control_hardware_type == 'real_hardware'}">
-                  <plugin>areumii_hardware_interface/AreumiiHardwareInterface</plugin>
-                </xacro:if>
-                <xacro:if value="${ros2_control_hardware_type == 'isaac'}">
+        <xacro:if value="${ros2_control_hardware_type == 'mock_components'}">
+          <ros2_control name="${name}" type="system">
+              <hardware>
+                <plugin>mock_components/GenericSystem</plugin>
+              </hardware>
+              <joint name="shoulder_pitch_joint_L">
+                  <command_interface name="position"/>
+                  <command_interface name="velocity"/>
+                  <state_interface name="position">
+                    <param name="initial_value">${initial_positions['shoulder_pitch_joint_L']}</param>
+                  </state_interface>
+                  <state_interface name="velocity"/>
+              </joint>
+              <joint name="shoulder_roll_joint_L">
+                  <command_interface name="position"/>
+                  <command_interface name="velocity"/>
+                  <state_interface name="position">
+                    <param name="initial_value">${initial_positions['shoulder_roll_joint_L']}</param>
+                  </state_interface>
+                  <state_interface name="velocity"/>
+              </joint>
+              <joint name="shouler_yaw_joint_L">
+                  <command_interface name="position"/>
+                  <command_interface name="velocity"/>
+                  <state_interface name="position">
+                    <param name="initial_value">${initial_positions['shouler_yaw_joint_L']}</param>
+                  </state_interface>
+                  <state_interface name="velocity"/>
+              </joint>
+              <joint name="elbow_joint_L">
+                  <command_interface name="position"/>
+                  <command_interface name="velocity"/>
+                  <state_interface name="position">
+                    <param name="initial_value">${initial_positions['elbow_joint_L']}</param>
+                  </state_interface>
+                  <state_interface name="velocity"/>
+              </joint>
+              <joint name="wrist_roll_joint_L">
+                  <command_interface name="position"/>
+                  <command_interface name="velocity"/>
+                  <state_interface name="position">
+                    <param name="initial_value">${initial_positions['wrist_roll_joint_L']}</param>
+                  </state_interface>
+                  <state_interface name="velocity"/>
+              </joint>
+              <joint name="wrist_yaw_joint_L">
+                  <command_interface name="position"/>
+                  <command_interface name="velocity"/>
+                  <state_interface name="position">
+                    <param name="initial_value">${initial_positions['wrist_yaw_joint_L']}</param>
+                  </state_interface>
+                  <state_interface name="velocity"/>
+              </joint>
+              <joint name="wrist_pitch_joint_L">
+                  <command_interface name="position"/>
+                  <command_interface name="velocity"/>
+                  <state_interface name="position">
+                    <param name="initial_value">${initial_positions['wrist_pitch_joint_L']}</param>
+                  </state_interface>
+                  <state_interface name="velocity"/>
+              </joint>
+              <joint name="shoulder_pitch_joint_R">
+                  <command_interface name="position"/>
+                  <command_interface name="velocity"/>
+                  <state_interface name="position">
+                    <param name="initial_value">${initial_positions['shoulder_pitch_joint_R']}</param>
+                  </state_interface>
+                  <state_interface name="velocity"/>
+              </joint>
+              <joint name="shoulder_roll_joint_R">
+                  <command_interface name="position"/>
+                  <command_interface name="velocity"/>
+                  <state_interface name="position">
+                    <param name="initial_value">${initial_positions['shoulder_roll_joint_R']}</param>
+                  </state_interface>
+                  <state_interface name="velocity"/>
+              </joint>
+              <joint name="shoulder_yaw_joint_R">
+                  <command_interface name="position"/>
+                  <command_interface name="velocity"/>
+                  <state_interface name="position">
+                    <param name="initial_value">${initial_positions['shoulder_yaw_joint_R']}</param>
+                  </state_interface>
+                  <state_interface name="velocity"/>
+              </joint>
+              <joint name="elbow_joint_R">
+                  <command_interface name="position"/>
+                  <command_interface name="velocity"/>
+                  <state_interface name="position">
+                    <param name="initial_value">${initial_positions['elbow_joint_R']}</param>
+                  </state_interface>
+                  <state_interface name="velocity"/>
+              </joint>
+              <joint name="wrist_roll_joint_R">
+                  <command_interface name="position"/>
+                  <command_interface name="velocity"/>
+                  <state_interface name="position">
+                    <param name="initial_value">${initial_positions['wrist_roll_joint_R']}</param>
+                  </state_interface>
+                  <state_interface name="velocity"/>
+              </joint>
+              <joint name="wrist_yaw_joint_R">
+                  <command_interface name="position"/>
+                  <command_interface name="velocity"/>
+                  <state_interface name="position">
+                    <param name="initial_value">${initial_positions['wrist_yaw_joint_R']}</param>
+                  </state_interface>
+                  <state_interface name="velocity"/>
+              </joint>
+              <joint name="wrist_pitch_joint_R">
+                  <command_interface name="position"/>
+                  <command_interface name="velocity"/>
+                  <state_interface name="position">
+                    <param name="initial_value">${initial_positions['wrist_pitch_joint_R']}</param>
+                  </state_interface>
+                  <state_interface name="velocity"/>
+              </joint>
+              <joint name="gripper_left_finger_joint_L">
+                  <command_interface name="position"/>
+                  <command_interface name="velocity"/>
+                  <state_interface name="position">
+                    <param name="initial_value">${initial_positions['gripper_left_finger_joint_L']}</param>
+                  </state_interface>
+                  <state_interface name="velocity"/>
+              </joint>
+              <joint name="gripper_right_finger_joint_L">
+                  <command_interface name="position"/>
+                  <command_interface name="velocity"/>
+                  <state_interface name="position">
+                    <param name="initial_value">${initial_positions['gripper_right_finger_joint_L']}</param>
+                  </state_interface>
+                  <state_interface name="velocity"/>
+              </joint>
+              <joint name="gripper_left_finger_joint_R">
+                  <command_interface name="position"/>
+                  <command_interface name="velocity"/>
+                  <state_interface name="position">
+                    <param name="initial_value">${initial_positions['gripper_left_finger_joint_R']}</param>
+                  </state_interface>
+                  <state_interface name="velocity"/>
+              </joint>
+              <joint name="gripper_right_finger_joint_R">
+                  <command_interface name="position"/>
+                  <command_interface name="velocity"/>
+                  <state_interface name="position">
+                    <param name="initial_value">${initial_positions['gripper_right_finger_joint_R']}</param>
+                  </state_interface>
+                  <state_interface name="velocity"/>
+              </joint>
+          </ros2_control>
+        </xacro:if>
+        <xacro:if value="${ros2_control_hardware_type == 'real_hardware'}">
+          <ros2_control name="${name}" type="system">
+              <hardware>
+                <plugin>areumii_hardware_interface/AreumiiHardwareInterface</plugin>
+              </hardware>
+              <joint name="shoulder_pitch_joint_L">
+                  <command_interface name="position"/>
+                  <command_interface name="velocity"/>
+                  <state_interface name="position">
+                    <param name="initial_value">${initial_positions['shoulder_pitch_joint_L']}</param>
+                  </state_interface>
+                  <state_interface name="velocity"/>
+              </joint>
+              <joint name="shoulder_roll_joint_L">
+                  <command_interface name="position"/>
+                  <command_interface name="velocity"/>
+                  <state_interface name="position">
+                    <param name="initial_value">${initial_positions['shoulder_roll_joint_L']}</param>
+                  </state_interface>
+                  <state_interface name="velocity"/>
+              </joint>
+              <joint name="shouler_yaw_joint_L">
+                  <command_interface name="position"/>
+                  <command_interface name="velocity"/>
+                  <state_interface name="position">
+                    <param name="initial_value">${initial_positions['shouler_yaw_joint_L']}</param>
+                  </state_interface>
+                  <state_interface name="velocity"/>
+              </joint>
+              <joint name="elbow_joint_L">
+                  <command_interface name="position"/>
+                  <command_interface name="velocity"/>
+                  <state_interface name="position">
+                    <param name="initial_value">${initial_positions['elbow_joint_L']}</param>
+                  </state_interface>
+                  <state_interface name="velocity"/>
+              </joint>
+              <joint name="wrist_roll_joint_L">
+                  <command_interface name="position"/>
+                  <command_interface name="velocity"/>
+                  <state_interface name="position">
+                    <param name="initial_value">${initial_positions['wrist_roll_joint_L']}</param>
+                  </state_interface>
+                  <state_interface name="velocity"/>
+              </joint>
+              <joint name="wrist_yaw_joint_L">
+                  <command_interface name="position"/>
+                  <command_interface name="velocity"/>
+                  <state_interface name="position">
+                    <param name="initial_value">${initial_positions['wrist_yaw_joint_L']}</param>
+                  </state_interface>
+                  <state_interface name="velocity"/>
+              </joint>
+              <joint name="wrist_pitch_joint_L">
+                  <command_interface name="position"/>
+                  <command_interface name="velocity"/>
+                  <state_interface name="position">
+                    <param name="initial_value">${initial_positions['wrist_pitch_joint_L']}</param>
+                  </state_interface>
+                  <state_interface name="velocity"/>
+              </joint>
+              <joint name="shoulder_pitch_joint_R">
+                  <command_interface name="position"/>
+                  <command_interface name="velocity"/>
+                  <state_interface name="position">
+                    <param name="initial_value">${initial_positions['shoulder_pitch_joint_R']}</param>
+                  </state_interface>
+                  <state_interface name="velocity"/>
+              </joint>
+              <joint name="shoulder_roll_joint_R">
+                  <command_interface name="position"/>
+                  <command_interface name="velocity"/>
+                  <state_interface name="position">
+                    <param name="initial_value">${initial_positions['shoulder_roll_joint_R']}</param>
+                  </state_interface>
+                  <state_interface name="velocity"/>
+              </joint>
+              <joint name="shoulder_yaw_joint_R">
+                  <command_interface name="position"/>
+                  <command_interface name="velocity"/>
+                  <state_interface name="position">
+                    <param name="initial_value">${initial_positions['shoulder_yaw_joint_R']}</param>
+                  </state_interface>
+                  <state_interface name="velocity"/>
+              </joint>
+              <joint name="elbow_joint_R">
+                  <command_interface name="position"/>
+                  <command_interface name="velocity"/>
+                  <state_interface name="position">
+                    <param name="initial_value">${initial_positions['elbow_joint_R']}</param>
+                  </state_interface>
+                  <state_interface name="velocity"/>
+              </joint>
+              <joint name="wrist_roll_joint_R">
+                  <command_interface name="position"/>
+                  <command_interface name="velocity"/>
+                  <state_interface name="position">
+                    <param name="initial_value">${initial_positions['wrist_roll_joint_R']}</param>
+                  </state_interface>
+                  <state_interface name="velocity"/>
+              </joint>
+              <joint name="wrist_yaw_joint_R">
+                  <command_interface name="position"/>
+                  <command_interface name="velocity"/>
+                  <state_interface name="position">
+                    <param name="initial_value">${initial_positions['wrist_yaw_joint_R']}</param>
+                  </state_interface>
+                  <state_interface name="velocity"/>
+              </joint>
+              <joint name="wrist_pitch_joint_R">
+                  <command_interface name="position"/>
+                  <command_interface name="velocity"/>
+                  <state_interface name="position">
+                    <param name="initial_value">${initial_positions['wrist_pitch_joint_R']}</param>
+                  </state_interface>
+                  <state_interface name="velocity"/>
+              </joint>
+          </ros2_control>
+          <ros2_control name="TEMPORARY_MOCK_gripper_system" type="system">
+              <hardware>
+                <plugin>mock_components/GenericSystem</plugin>
+              </hardware>
+              <joint name="gripper_left_finger_joint_L">
+                  <command_interface name="position"/>
+                  <command_interface name="velocity"/>
+                  <state_interface name="position">
+                    <param name="initial_value">${initial_positions['gripper_left_finger_joint_L']}</param>
+                  </state_interface>
+                  <state_interface name="velocity"/>
+              </joint>
+              <joint name="gripper_right_finger_joint_L">
+                  <command_interface name="position"/>
+                  <command_interface name="velocity"/>
+                  <state_interface name="position">
+                    <param name="initial_value">${initial_positions['gripper_right_finger_joint_L']}</param>
+                  </state_interface>
+                  <state_interface name="velocity"/>
+              </joint>
+              <joint name="gripper_left_finger_joint_R">
+                  <command_interface name="position"/>
+                  <command_interface name="velocity"/>
+                  <state_interface name="position">
+                    <param name="initial_value">${initial_positions['gripper_left_finger_joint_R']}</param>
+                  </state_interface>
+                  <state_interface name="velocity"/>
+              </joint>
+              <joint name="gripper_right_finger_joint_R">
+                  <command_interface name="position"/>
+                  <command_interface name="velocity"/>
+                  <state_interface name="position">
+                    <param name="initial_value">${initial_positions['gripper_right_finger_joint_R']}</param>
+                  </state_interface>
+                  <state_interface name="velocity"/>
+              </joint>
+          </ros2_control>
+        </xacro:if>
+        <xacro:if value="${ros2_control_hardware_type == 'isaac'}">
+          <ros2_control name="${name}" type="system">
+              <hardware>
                   <plugin>topic_based_ros2_control/TopicBasedSystem</plugin>
                   <param name="joint_commands_topic">/isaac_joint_commands</param>
                   <param name="joint_states_topic">/isaac_joint_states</param>
-                </xacro:if>
-            </hardware>
-            <joint name="shoulder_pitch_joint_L">
-                <command_interface name="position"/>
-                <command_interface name="velocity"/>
-                <state_interface name="position">
-                  <param name="initial_value">${initial_positions['shoulder_pitch_joint_L']}</param>
-                </state_interface>
-                <state_interface name="velocity"/>
-            </joint>
-            <joint name="shoulder_roll_joint_L">
-                <command_interface name="position"/>
-                <command_interface name="velocity"/>
-                <state_interface name="position">
-                  <param name="initial_value">${initial_positions['shoulder_roll_joint_L']}</param>
-                </state_interface>
-                <state_interface name="velocity"/>
-            </joint>
-            <joint name="shouler_yaw_joint_L">
-                <command_interface name="position"/>
-                <command_interface name="velocity"/>
-                <state_interface name="position">
-                  <param name="initial_value">${initial_positions['shouler_yaw_joint_L']}</param>
-                </state_interface>
-                <state_interface name="velocity"/>
-            </joint>
-            <joint name="elbow_joint_L">
-                <command_interface name="position"/>
-                <command_interface name="velocity"/>
-                <state_interface name="position">
-                  <param name="initial_value">${initial_positions['elbow_joint_L']}</param>
-                </state_interface>
-                <state_interface name="velocity"/>
-            </joint>
-            <joint name="wrist_roll_joint_L">
-                <command_interface name="position"/>
-                <command_interface name="velocity"/>
-                <state_interface name="position">
-                  <param name="initial_value">${initial_positions['wrist_roll_joint_L']}</param>
-                </state_interface>
-                <state_interface name="velocity"/>
-            </joint>
-            <joint name="wrist_yaw_joint_L">
-                <command_interface name="position"/>
-                <command_interface name="velocity"/>
-                <state_interface name="position">
-                  <param name="initial_value">${initial_positions['wrist_yaw_joint_L']}</param>
-                </state_interface>
-                <state_interface name="velocity"/>
-            </joint>
-            <joint name="wrist_pitch_joint_L">
-                <command_interface name="position"/>
-                <command_interface name="velocity"/>
-                <state_interface name="position">
-                  <param name="initial_value">${initial_positions['wrist_pitch_joint_L']}</param>
-                </state_interface>
-                <state_interface name="velocity"/>
-            </joint>
-            <joint name="shoulder_pitch_joint_R">
-                <command_interface name="position"/>
-                <command_interface name="velocity"/>
-                <state_interface name="position">
-                  <param name="initial_value">${initial_positions['shoulder_pitch_joint_R']}</param>
-                </state_interface>
-                <state_interface name="velocity"/>
-            </joint>
-            <joint name="shoulder_roll_joint_R">
-                <command_interface name="position"/>
-                <command_interface name="velocity"/>
-                <state_interface name="position">
-                  <param name="initial_value">${initial_positions['shoulder_roll_joint_R']}</param>
-                </state_interface>
-                <state_interface name="velocity"/>
-            </joint>
-            <joint name="shoulder_yaw_joint_R">
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