Commit message: feat: dgl_ros 를 통해 grasp_poses 후보들 생성 완료. ros2 control 을 아이작, CAN 통신, mock 각각에 대해서 분기문으로 수정. C1 URDF joint 축들을 거울 상으로 다시 배치 함. actor.hpp 은 dgl_ros 액션 서버가 SUCCEED 상태로 반환 되도록 코드를 수정함.

File: src/areumii_description/urdf/areumii.xacro (robot description, xacro)
@@ -433,5 +433,5 @@
   <parent link="shoulder_roll_link_L_1"/>
   <child link="shoulder_yaw_link_L_1"/>
-  <axis xyz="0.0 0.0 1.0"/>
+  <axis xyz="0.0 0.0 -1.0"/>
   <limit upper="1.396263" lower="-1.396263" effort="100" velocity="100"/>
 </joint>
@@ -440,6 +440,6 @@
   <parent link="shoulder_yaw_link_L_1"/>
   <child link="elbow_link_L_1"/>
-  <axis xyz="0.0 1.0 -0.0"/>
-  <limit upper="0.872665" lower="-2.094395" effort="100" velocity="100"/>
+  <axis xyz="0.0 -1.0 -0.0"/>
+  <limit upper="2.094395" lower="-0.872665" effort="100" velocity="100"/>
 </joint>
 <joint name="wrist_roll_joint_L" type="revolute">
@@ -447,5 +447,5 @@
   <parent link="elbow_link_L_1"/>
   <child link="wrist_roll_link_L_1"/>
-  <axis xyz="0.0 0.0 1.0"/>
+  <axis xyz="0.0 0.0 -1.0"/>
   <limit upper="1.745329" lower="-1.745329" effort="100" velocity="100"/>
 </joint>
@@ -454,5 +454,5 @@
   <parent link="wrist_roll_link_L_1"/>
   <child link="wrist_yaw_link_L_1"/>
-  <axis xyz="1.0 -0.0 0.0"/>
+  <axis xyz="-1.0 -0.0 0.0"/>
   <limit upper="0.523599" lower="-0.523599" effort="100" velocity="100"/>
 </joint>
@@ -461,5 +461,5 @@
   <parent link="wrist_yaw_link_L_1"/>
   <child link="wrist_pitch_link_L_1"/>
-  <axis xyz="0.0 1.0 -0.0"/>
+  <axis xyz="0.0 -1.0 -0.0"/>
   <limit upper="1.570796" lower="-1.570796" effort="100" velocity="100"/>
 </joint>
@@ -475,6 +475,6 @@
   <parent link="shoulder_yaw_link_R_1"/>
   <child link="elbow_link_R_1"/>
-  <axis xyz="0.0 1.0 -0.0"/>
-  <limit upper="0.872665" lower="-2.094395" effort="100" velocity="100"/>
+  <axis xyz="0.0 -1.0 -0.0"/>
+  <limit upper="2.094395" lower="-0.872665" effort="100" velocity="100"/>
 </joint>
 <joint name="wrist_roll_joint_R" type="revolute">
@@ -496,5 +496,5 @@
   <parent link="wrist_yaw_link_R_1"/>
   <child link="wrist_pitch_link_R_1"/>
-  <axis xyz="0.0 1.0 -0.0"/>
+  <axis xyz="0.0 -1.0 -0.0"/>
   <limit upper="1.570796" lower="-1.570796" effort="100" velocity="100"/>
 </joint>
@@ -503,6 +503,6 @@
   <parent link="shoulder_pitch_link_R_1"/>
   <child link="shoulder_roll_link_R_1"/>
-  <axis xyz="1.0 -0.0 0.0"/>
-  <limit upper="0.261799" lower="-2.96706" effort="100" velocity="100"/>
+  <axis xyz="-1.0 -0.0 0.0"/>
+  <limit upper="2.96706" lower="-0.261799" effort="100" velocity="100"/>
 </joint>
 <joint name="shoulder_pitch_joint_R" type="revolute">

Commit message: feat: MTC 로 왼손 그리퍼 제어 성공. 이 과정에서 URDF 및 Xacro 에 mimic 추가함. moveit_controllers.yaml 에도 command interface 를 수정함.

File: src/areum_ii_moveit_config/config/areumii.ros2_control.xacro (robot description, xacro)
@@ -129,6 +129,6 @@
               </joint>
               <joint name="gripper_right_finger_joint_L">
-                  <command_interface name="position"/>
-                  <command_interface name="velocity"/>
+                  <param name="mimic">gripper_left_finger_joint_L</param>
+                  <param name="multiplier">-1.0</param>
                   <state_interface name="position">
                     <param name="initial_value">${initial_positions['gripper_right_finger_joint_L']}</param>

File: src/areumii_description/urdf/areumii.urdf (robot description, URDF)
Before this commit: robot areumii, 22 links, 21 joints
Joints:
- joint gripper_right_finger_joint_L: mimic (none) -> joint=gripper_left_finger_joint_L multiplier=-1.0 offset=0.0
- joint gripper_right_finger_joint_R: mimic (none) -> joint=gripper_left_finger_joint_R multiplier=-1.0 offset=0.0

File: src/areumii_description/urdf/areumii.xacro (robot description, xacro)
@@ -533,4 +533,5 @@
   <axis xyz="0.0 1.0 -0.0"/>
   <limit upper="0.0" lower="-0.03" effort="100" velocity="100"/>
+  <mimic joint="gripper_left_finger_joint_L" multiplier="-1.0" offset="0.0"/>
 </joint>
 <joint name="gripper_hand_joint_L" type="fixed">
@@ -552,4 +553,5 @@
   <axis xyz="0.0 1.0 -0.0"/>
   <limit upper="0.0" lower="-0.03" effort="100" velocity="100"/>
+  <mimic joint="gripper_left_finger_joint_R" multiplier="-1.0" offset="0.0"/>
 </joint>
 <joint name="gripper_hand_joint_R" type="fixed">

Commit message: feat: Pick and Place Deploy 시도 >> 움직이긴 하나, gpd_config 방향필터 조정 해야함

File: src/areum_ii_moveit_config/config/areumii.ros2_control.xacro (robot description, xacro)
@@ -215,4 +215,12 @@
                   <state_interface name="velocity"/>
               </joint>
+              <joint name="gripper_left_finger_joint_L">
+                  <command_interface name="position"/>
+                  <command_interface name="velocity"/>
+                  <state_interface name="position">
+                    <param name="initial_value">${initial_positions['gripper_left_finger_joint_L']}</param>
+                  </state_interface>
+                  <state_interface name="velocity"/>
+              </joint>
               <joint name="shoulder_pitch_joint_R">
                   <command_interface name="position"/>
@@ -271,25 +279,4 @@
                   <state_interface name="velocity"/>
               </joint>
-          </ros2_control>
-          <ros2_control name="TEMPORARY_MOCK_gripper_system" type="system">
-              <hardware>
-                <plugin>mock_components/GenericSystem</plugin>
-              </hardware>
-              <joint name="gripper_left_finger_joint_L">
-                  <command_interface name="position"/>
-                  <command_interface name="velocity"/>
-                  <state_interface name="position">
-                    <param name="initial_value">${initial_positions['gripper_left_finger_joint_L']}</param>
-                  </state_interface>
-                  <state_interface name="velocity"/>
-              </joint>
-              <joint name="gripper_right_finger_joint_L">
-                  <command_interface name="position"/>
-                  <command_interface name="velocity"/>
-                  <state_interface name="position">
-                    <param name="initial_value">${initial_positions['gripper_right_finger_joint_L']}</param>
-                  </state_interface>
-                  <state_interface name="velocity"/>
-              </joint>
               <joint name="gripper_left_finger_joint_R">
                   <command_interface name="position"/>
@@ -297,12 +284,4 @@
                   <state_interface name="position">
                     <param name="initial_value">${initial_positions['gripper_left_finger_joint_R']}</param>
-                  </state_interface>
-                  <state_interface name="velocity"/>
-              </joint>
-              <joint name="gripper_right_finger_joint_R">
-                  <command_interface name="position"/>
-                  <command_interface name="velocity"/>
-                  <state_interface name="position">
-                    <param name="initial_value">${initial_positions['gripper_right_finger_joint_R']}</param>
                   </state_interface>
                   <state_interface name="velocity"/>
